Commit message: feat(vision): M3检测框3D投影节点detection_marker
- 新增detection_marker.py: Detection2DArray→MarkerArray(LINE_STRIP框+文字标签)
- 针孔模型投影到固定深度平面, lifetime 0.5s自动过期, 类别crc32配色
- URDF补camera_optical_link固定关节(REP103 rpy=-pi/2 0 -pi/2)
- camera yaml frame_id改camera_optical_link; yolo.yaml加内参段
- setup.py加入口, package.xml加visualization_msgs, launch三节点齐发

File: xuegecar_description/urdf/leap_ros.urdf (robot description, URDF)
Before this commit: robot xuegecar, 14 links, 13 joints
Links:
- added link camera_optical_link
Joints:
- added joint camera_optical_joint: type fixed, parent camera_link, child camera_optical_link, origin xyz=0 0 0 rpy=-1.57079632679 0 -1.57079632679
